File: 2. VL53L5CX/Swift_Module_VL53L5CX.kicad_pcb (KiCad board)
At the start: 4 copper layers, 38.8 x 18.8 mm, 19 parts, among them IC2 VL53L5CXV0GC_1, J1 5V_In, J2 Conn_01x12_MountingPin, J3 Conn_01x07, U1 XC6206P332MR

Commit message: I forgor
Parts:
- removed REF**: OSHW-Logo_5.7x6mm_SilkScreen, Symbol:OSHW-Logo_5.7x6mm_SilkScreen
- J3: footprint Connector_PinHeader_1.00mm:PinHeader_1x07_P1.00mm_Vertical -> Connector_PinHeader_2.54mm:PinHeader_1x07_P2.54mm_Vertical
- moved J3 0.31 mm to (121.0, 53.6)
Routing:
- net /I2C_RST: track 22.3 -> 27.2 mm
- net /GPIO: track 20.1 -> 22.6 mm
- net /SDA: track 22.4 -> 23.4 mm
- net /SCL: track 24.8 -> 25.5 mm
- net /INT: track 20.4 -> 20.3 mm, vias 2 -> 3
- net GND: vias 92 -> 93
