File: 2. VL53L5CX/Swift_Module_VL53L5CX.kicad_sch (KiCad schematic)
At the start: 19 parts, among them IC2 VL53L5CXV0GC_1, J1 5V_In, J2 Conn_01x12_MountingPin, J3 Conn_01x07, U1 XC6206P332MR

Commit message: I forgor
Parts:
- J3: footprint Connector_PinHeader_1.00mm:PinHeader_1x07_P1.00mm_Vertical -> Connector_PinHeader_2.54mm:PinHeader_1x07_P2.54mm_Vertical
Changed lines of the file:
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@@
 			)
 		)
-		(property "Footprint" "Connector_PinHeader_1.00mm:PinHeader_1x07_P1.00mm_Vertical"
+		(property "Footprint" "Connector_PinHeader_2.54mm:PinHeader_1x07_P2.54mm_Vertical"
 			(at 163.195 107.95 0)
 			(effects
